Commit message: Added Velodyne VLP16 to the Husky simulator

File: husky_description/urdf/husky.urdf.xacro (robot description, xacro)
@@ -29,4 +29,5 @@
   <xacro:include filename="$(find husky_description)/urdf/accessories/sensor_arch.urdf.xacro"/>
   <xacro:include filename="$(find ur_description)/urdf/ur5.urdf.xacro" />
+  <xacro:include filename="$(find velodyne_description)/urdf/VLP-16.urdf.xacro" />
   <property name="M_PI" value="3.14159"/>
   <!-- Base Size -->
@@ -126,4 +127,7 @@
         <child link="base_laser_mount" />
       </joint>
+      <xacro:VLP-16 parent="top_plate_link" name="vlp" topic="vlp">
+        <origin xyz="0.25 0 0.1765" rpy="0.0 0.0 0.0" />
+      </xacro:VLP-16>
     </xacro:if>
     <xacro:if value="$(arg kinect_enabled)">
@@ -134,7 +138,7 @@
         <origin xyz="$(optenv HUSKY_KINECT_XYZ 0 0 0)" rpy="$(optenv HUSKY_KINECT_RPY 0 0.18 3.14)" />
         <parent link="sensor_arch_mount_link"/>
-        <child link="camera_link"/>
+        <child link="kinect_link"/>
       </joint>
-      <xacro:kinect_camera prefix="camera"/>
+      <xacro:kinect_camera prefix="kinect"/>
     </xacro:if>
   </xacro:macro>
